File: NGI_Battery_simulator_adapter.kicad_sch (KiCad schematic)
At the start: 31 parts, among them J1 Screw_Terminal_01x20, J2 1725042, J3 Conn_01x05, J4 Screw_Terminal_01x20, J6 1725042

Commit message: gerber update
fix some DRC error, minor change
Other:
- note added: "Mounting holes"
- note added: "pin 1 and pin 2 .... pin 23 and pin 24 shorted on connector,"
- moved on the sheet: J2, J6, R1, R2, R3, R4, R5, R6, R7, R8
